Commit message: feat: add scan filter node, add left and right distance sensors in URDF, and configure Nav2 costmaps

File: models/nebula_urdf/gazebo_plugins.xacro (robot description, xacro)
@@ -106,4 +106,64 @@
     </sensor>
   </gazebo>
+  <!-- ===== Sol Ön Mesafe Sensörü (Ray Sensor) ===== -->
+  <gazebo reference="left_sensor_link">
+    <sensor type="ray" name="left_distance_sensor">
+      <pose>0 0 0 0 0 0</pose>
+      <visualize>true</visualize>
+      <update_rate>10.0</update_rate>
+      <ray>
+        <scan>
+          <horizontal>
+            <samples>1</samples>
+            <resolution>1</resolution>
+            <min_angle>-0.01</min_angle>
+            <max_angle>0.01</max_angle>
+          </horizontal>
+        </scan>
+        <range>
+          <min>0.05</min>
+          <max>3.0</max>
+          <resolution>0.01</resolution>
+        </range>
+      </ray>
+      <plugin name="gazebo_ros_left_sensor" filename="libgazebo_ros_ray_sensor.so">
+        <ros>
+          <remapping>~/out:=/left_sensor/scan</remapping>
+        </ros>
+        <output_type>sensor_msgs/LaserScan</output_type>
+        <frame_name>left_sensor_link</frame_name>
+      </plugin>
+    </sensor>
+  </gazebo>
+  <!-- ===== Sağ Ön Mesafe Sensörü (Ray Sensor) ===== -->
+  <gazebo reference="right_sensor_link">
+    <sensor type="ray" name="right_distance_sensor">
+      <pose>0 0 0 0 0 0</pose>
+      <visualize>true</visualize>
+      <update_rate>10.0</update_rate>
+      <ray>
+        <scan>
+          <horizontal>
+            <samples>1</samples>
+            <resolution>1</resolution>
+            <min_angle>-0.01</min_angle>
+            <max_angle>0.01</max_angle>
+          </horizontal>
+        </scan>
+        <range>
+          <min>0.05</min>
+          <max>3.0</max>
+          <resolution>0.01</resolution>
+        </range>
+      </ray>
+      <plugin name="gazebo_ros_right_sensor" filename="libgazebo_ros_ray_sensor.so">
+        <ros>
+          <remapping>~/out:=/right_sensor/scan</remapping>
+        </ros>
+        <output_type>sensor_msgs/LaserScan</output_type>
+        <frame_name>right_sensor_link</frame_name>
+      </plugin>
+    </sensor>
+  </gazebo>
   <!-- ===== IMU Sensör Eklentisi ===== -->
   <gazebo reference="imu_link">

File: models/nebula_urdf/model.xacro (robot description, xacro)
@@ -180,4 +180,25 @@
   <xacro:LIDAR x="0" y="0" z="0.2"/>
   <xacro:IMU x="0" y="0" z="0.09"/>
+  <!-- DISTANCE SENSOR MACRO -->
+  <xacro:macro name="DISTANCE_SENSOR" params="name x y z">
+    <link name="${name}_link">
+      <xacro:box_inertia m="0.01" l="0.02" w="0.02" h="0.02" xyz="0 0 0" rpy="0 0 0"/>
+      <visual>
+        <geometry><box size="0.02 0.02 0.02"/></geometry>
+        <material name="white"><color rgba="1 1 1 1"/></material>
+      </visual>
+      <collision>
+        <geometry><box size="0.02 0.02 0.02"/></geometry>
+      </collision>
+    </link>
+    <joint name="${name}_joint" type="fixed">
+      <parent link="base_link"/>
+      <child link="${name}_link"/>
+      <origin xyz="${x} ${y} ${z}" rpy="0 0 0"/>
+    </joint>
+  </xacro:macro>
+  <!-- Front Distance Sensors (placed in front of the left/right columns) -->
+  <xacro:DISTANCE_SENSOR name="left_sensor" x="0.431" y="0.12" z="0.2"/>
+  <xacro:DISTANCE_SENSOR name="right_sensor" x="0.431" y="-0.12" z="0.2"/>
   <!-- ============================================================ -->
   <!-- FORKLİFT KALDIRMA MEKANİZMASI (DETACHABLE / AYRILABİLİR) -->

Commit message: style: sanitize remaining model comments and material definitions

File: models/nebula_urdf/gazebo_plugins.xacro (robot description, xacro)
@@ -16,7 +16,7 @@
     <material>Gazebo/White</material>
   </gazebo>
-  <!-- Yan panel: SIRIUS dokulu material (scripts/sirius.material) -->
+  <!-- Yan panel: NEBULA dokulu material (scripts/nebula.material) -->
   <gazebo reference="left_panel_link">
-    <material>Sirius/Label</material>
+    <material>Nebula/Label</material>
   </gazebo>
   <gazebo reference="left_wheel_link">

File: models/nebula_urdf/model.xacro (robot description, xacro)
@@ -48,5 +48,5 @@
     <child link="front_marker_link"/>
   </joint>
-  <!-- YAN PANEL — sol yüze (+Y) "SIRIUS" yazılı doku -->
+  <!-- YAN PANEL — sol yüze (+Y) "NEBULA" yazılı doku -->
   <material name="nebula_label">
     <texture filename="package://amr_forklift/models/nebula_urdf/materials/textures/nebula_label.png"/>

File: models/nebula_urdf/properties.xacro (robot description, xacro)
@@ -1,4 +1,4 @@
 <?xml version = "1.0"?>
-<robot name = "sirius" xmlns:xacro="http://www.ros.org/wiki/xacro">
+<robot name = "nebula" xmlns:xacro="http://www.ros.org/wiki/xacro">
     <xacro:macro name = "box_inertia" params = "m l w h xyz rpy">
         <inertial>

File: models/nebula_urdf/ros2_controller.xacro (robot description, xacro)
@@ -1,7 +1,7 @@
 <?xml version="1.0"?>
 <robot xmlns:xacro="http://ros.org/wiki/xacro">
-<ros2_control name="SiriusHardware" type="system">
+<ros2_control name="NebulaHardware" type="system">
   <hardware>
-    <plugin>SiriusHardware</plugin>
+    <plugin>NebulaHardware</plugin>
     <param name="device">/dev/ttyACM0</param>
     <param name="baud_rate">115200</param>
